File: kicad/little-clocky/inputs.kicad_sch (KiCad schematic)
At the start: 29 parts, among them CN1 WQP518MA, CN2 WQP518MA, CN3 WQP518MA, CN4 WQP518MA, CN5 WQP518MA, CN6 WQP518MA, Q1 NPN, Q2 NPN, SW1 RotaryEncoder_Switch, SW2 SW_Push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

Commit message: like 5 different PCB refreshes
Connections:
- net TRIG1: now also Q2.1 (C), R35.1; no longer Q1.1 (C), R34.1
- net TRIG2: now also Q1.1 (C), R34.1; no longer Q2.1 (C), R35.1
Changed lines of the file:
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@@
-		)
-	)
-	(global_label "TRIG1"
-		(shape output)
-		(at 154.94 49.53 0)
-		(fields_autoplaced yes)
-		(effects
-			(font
-				(size 1.27 1.27)
-			)
-			(justify left)
-		)
-		(property "Intersheetrefs" "${INTERSHEET_REFS}"
-			(at 163.2471 49.53 0)
-			(hide yes)
-			(show_name no)
-			(do_not_autoplace no)
-			(effects
-				(font
-					(size 1.27 1.27)
-				)
-				(justify left)
-			)
-		)
-	)
-	(global_label "TRIG2"
-		(shape output)
-		(at 156.21 105.41 0)
-		(fields_autoplaced yes)
-		(effects
-			(font
-				(size 1.27 1.27)
-			)
-			(justify left)
-		)
-		(property "Intersheetrefs" "${INTERSHEET_REFS}"
-			(at 164.5171 105.41 0)
-			(hide yes)
-			(show_name no)
-			(do_not_autoplace no)
-			(effects
-				(font
-					(size 1.27 1.27)
-				)
-				(justify left)
-			)
 		)
 	)
@@
 				)
 				(justify right)
+			)
+		)
+	)
+	(global_label "TRIG2"
+		(shape output)
+		(at 154.94 49.53 0)
+		(fields_autoplaced yes)
+		(effects
+			(font
+				(size 1.27 1.27)
+			)
+			(justify left)
+		)
+		(property "Intersheetrefs" "${INTERSHEET_REFS}"
+			(at 163.2471 49.53 0)
+			(hide yes)
+			(show_name no)
+			(do_not_autoplace no)
+			(effects
+				(font
+					(size 1.27 1.27)
+				)
+				(justify left)
 			)
 		)
@@
 			(hide yes)
 			(show_name no)
+			(do_not_autoplace no)
+			(effects
+				(font
+					(size 1.27 1.27)
+				)
+				(justify left)
+			)
+		)
+	)
+	(global_label "TRIG1"
+		(shape output)
+		(at 156.21 105.41 0)
+		(fields_autoplaced yes)
+		(effects
+			(font
+				(size 1.27 1.27)
+			)
+			(justify left)
+		)
+		(property "Intersheetrefs" "${INTERSHEET_REFS}"
+			(at 164.5171 105.41 0)
+			(hide yes)
+			(show_name no)
