File: kicad/little-clocky/little-clocky.kicad_pcb (KiCad board)
At the start: 2 copper layers, 45 x 100 mm, 63 parts, among them CN1 WQP518MA, CN2 WQP518MA, CN3 WQP518MA, CN4 WQP518MA, CN5 WQP518MA, CN6 WQP518MA, J1 Conn_02x05_Odd_Even, J2 WQP518MA, J3 WQP518MA, J4 WQP518MA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

Commit message: beat magic
Parts:
- moved R16 84.9 mm to (119.4, 100.1), turned to 90 degrees
- moved R1 84.0 mm to (120.4, 86.4), turned to 0 degrees
- moved R4 82.5 mm to (120.4, 94.0), turned to 0 degrees
- moved R15 82.3 mm to (115.8, 100.1), turned to 90 degrees
- moved R14 80.0 mm to (112.3, 100.1), turned to 90 degrees
- moved R11 78.0 mm to (105.2, 100.1), turned to 90 degrees
- moved R6 77.6 mm to (119.4, 82.3), turned to 90 degrees
- moved R5 74.2 mm to (115.8, 80.3), turned to -90 degrees
- moved R12 73.0 mm to (101.6, 100.1), turned to 90 degrees
- moved R7 70.3 mm to (112.3, 82.3), turned to 90 degrees
- moved R9 70.0 mm to (101.6, 80.3), turned to -90 degrees
- moved R13 69.5 mm to (98.0, 100.1), turned to 90 degrees
- moved R10 66.0 mm to (98.0, 82.3), turned to 90 degrees
- moved R8 63.2 mm to (105.2, 82.3), turned to 90 degrees
- moved R3 63.0 mm to (97.5, 94.0)
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Routing:
- net Net-(R1-Pad1): track 21.3 -> 0.00 mm

Commit message: like 5 different PCB refreshes
Parts:
- added R29: 470, Resistor_THT:R_Axial_DIN0309_L9.0mm_D3.2mm_P2.54mm_Vertical, B.Cu at (67.4, 128.2)
- D1, D2, U4: moved to F.Cu
- moved R6 75.9 mm to (46.7, 104.1), turned to 0 degrees
- moved R15 71.4 mm to (52.8, 66.5), turned to 0 degrees
- moved U3 71.1 mm to (47.2, 69.6), turned to 0 degrees
- moved R1 70.4 mm to (52.3, 104.1)
- moved R5 67.9 mm to (49.3, 66.5), turned to 180 degrees
- moved C4 60.9 mm to (50.8, 80.3)
- moved R14 59.6 mm to (65.5, 63.0)
- moved C3 58.4 mm to (50.8, 74.1)
- moved R9 54.9 mm to (47.2, 87.9)
- moved R7 53.9 mm to (65.5, 55.4), turned to -90 degrees
- moved R24 51.9 mm to (85.3, 66.5), turned to 0 degrees
- moved R11 51.9 mm to (71.1, 61.0), turned to 180 degrees
- moved R12 47.8 mm to (54.9, 89.9)
- moved R21 47.1 mm to (81.8, 66.5), turned to 180 degrees
- moved R10 45.7 mm to (57.9, 104.1), turned to 0 degrees
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Routing:
- net AREF_-10V: track 0.00 -> 113.9 mm
- net +12V: track 0.00 -> 109.5 mm, vias 0 -> 2
- net ENCS: track 0.00 -> 105.4 mm
- net ENCA: track 0.00 -> 75.3 mm, vias 0 -> 2
- net ENCB: track 0.00 -> 74.9 mm
- net +3.3V: track 0.00 -> 74.2 mm, vias 0 -> 1
- net -12V: track 0.00 -> 71.0 mm, vias 0 -> 1
- net BTN2: track 0.00 -> 70.8 mm
- net +5V: track 0.00 -> 68.9 mm, vias 0 -> 3
- net BTN1: track 0.00 -> 65.4 mm
- net Net-(U4C--): track 0.00 -> 65.2 mm
- net Net-(U4A--): track 0.00 -> 63.6 mm
- net Net-(U3D--): track 0.00 -> 58.3 mm
- net Net-(R16-Pad2): track 0.00 -> 53.8 mm
- net Net-(U4D--): track 0.00 -> 50.8 mm
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- added copper zone on B.Cu, net GND
- added copper zone on F.Cu, net GND
Other:
- board size 45 x 100 mm -> 45.5 x 100 mm
