File: kicad/little-clocky/little-clocky.kicad_sch (KiCad schematic)
At the start: 12 parts, among them J1 Conn_02x05_Odd_Even, U2 AZ1117-5.0, U5 LM4040DBZ-10

Commit message: like 5 different PCB refreshes
Parts:
- R29: footprint (none) -> Resistor_THT:R_Axial_DIN0309_L9.0mm_D3.2mm_P2.54mm_Vertical
Changed lines of the file:
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@@
 			)
 		)
-		(property "Footprint" ""
+		(property "Footprint" "Resistor_THT:R_Axial_DIN0309_L9.0mm_D3.2mm_P2.54mm_Vertical"
 			(at 234.442 35.56 90)
 			(hide yes)
